File: Power Systems.kicad_sch (KiCad schematic)
At the start: 0 parts

Commit message: Battery Block
Stage 1 - Battery Block
Parts:
- added BT1: 6S LiPo 22.2V 9000mAh, Package_SON:Texas_DRC0010J_ThermalVias, symbol Device:Battery
- added C1: 1000 uF 35V, symbol Device:C_Polarized
- added D1: D_Schottky, symbol Device:D_Schottky
- added F1: 25A FUSE, Package_LCC:PLCC-84_29.3x29.3mm_P1.27mm, symbol Device:Fuse
- added J1: CURRENT SENSE, symbol Connector_Generic:Conn_01x03
- added K1: E-STOP RELAY 30A, Relay_THT:Relay_SPDT_SANYOU_SRD_Series_Form_C, symbol Relay:SANYOU_SRD_Form_C
- added SW1: MAIN DISCONECT - 30A, Button_Switch_THT:SW_NKK_GW12LJP, symbol Switch:SW_SPST
- added SW2: E-STOP NC, Button_Switch_THT:SW_NKK_GW12LJP, symbol Switch:SW_DPST
Connections:
- new net: BT1.1 (+), SW1.1 (A)
- new net: F1.1, SW1.2 (B)
- new net: D1.2 (A), F1.2
- new net GND: BT1.2 (-), C1.2
- new net VBATT: C1.1, D1.1 (K)
Other:
- company: (none) -> University of Colorado Boulder
- title: (none) -> Rover Electrical Power Systems
