File: Power Systems/Power Systems.kicad_sch (KiCad schematic)
At the start: 8 parts, among them J1 CURRENT SENSE, K1 E-STOP RELAY 30A, SW1 MAIN DISCONECT - 30A, SW2 E-STOP NC

Commit message: Restructure
(Open _sch file only for now)
Parts:
- added F2, F3, F4, F5: 7.5 ATO, Package_LCC:PLCC-84_29.3x29.3mm_P1.27mm, symbol Device:Fuse
- added J2: Conn_01x02, symbol Connector_Generic:Conn_01x02

Commit message: Motor Driver
Parts:
- added J2: MOTOR DRIVER 2, symbol Connector_Generic:Conn_01x02
- added J3: MOTOR DRIVER 3, symbol Connector_Generic:Conn_01x02
- added J4: MOTOR DRIVER 4, symbol Connector_Generic:Conn_01x02
- J1: renamed from J2; value Conn_01x02 -> MOTOR DRIVER 1
Changed lines of the file:
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@@
+	)
+	(symbol
+		(lib_id "Connector_Generic:Conn_01x02")
+		(at 185.42 97.79 0)
+		(unit 1)
+		(body_style 1)
+		(exclude_from_sim no)
+		(in_bom yes)
+		(on_board yes)
+		(in_pos_files yes)
+		(dnp no)
+		(fields_autoplaced yes)
+		(property "Reference" "J3"
+			(at 187.96 97.7899 0)
+			(show_name no)
+			(do_not_autoplace no)
+			(effects
+				(font
+					(size 1.27 1.27)
+				)
+				(justify left)
+			)
+		)
+		(property "Value" "MOTOR DRIVER 3"
+			(at 187.96 100.3299 0)
+			(show_name no)
+			(do_not_autoplace no)
+			(effects
+				(font
+					(size 1.27 1.27)
+				)
+				(justify left)
+			)
+		)
+		(property "Footprint" ""
+			(at 185.42 97.79 0)
+			(hide yes)
+			(show_name no)
+			(do_not_autoplace no)
+			(effects
+				(font
+					(size 1.27 1.27)
+				)
+			)
+		)
+		(property "Datasheet" ""
+			(at 185.42 97.79 0)
+			(hide yes)
+			(show_name no)
+			(do_not_autoplace no)
+			(effects
+				(font
+					(size 1.27 1.27)
+				)
+			)
+		)
+		(property "Description" "Generic connector, single row, 01x02, script generated (kicad-library-utils/schlib/autogen/connector/)"
+			(at 185.42 97.79 0)
+			(hide yes)
+			(show_name no)
+			(do_not_autoplace no)
+			(effects
+				(font
+					(size 1.27 1.27)
+				)
+			)
+		)
+		(pin "1"
+		)
+		(pin "2"
+		)
+		(instances
+			(project "Power Systems"
+				(path "/7d9b4746-b4fa-4905-9b55-f00e27d57e0a"
+					(reference "J3")
+					(unit 1)
+				)
+			)
+		)
 	)
 	(symbol
@@
 	)
 	(symbol
+		(lib_id "Connector_Generic:Conn_01x02")
+		(at 185.42 90.17 0)
+		(unit 1)
+		(body_style 1)
+		(exclude_from_sim no)
+		(in_bom yes)
+		(on_board yes)
+		(in_pos_files yes)
+		(dnp no)
+		(fields_autoplaced yes)
+		(property "Reference" "J2"
+			(at 187.96 90.1699 0)
+			(show_name no)
+			(do_not_autoplace no)
+			(effects
+				(font
+					(size 1.27 1.27)
+				)
+				(justify left)
+			)
+		)
+		(property "Value" "MOTOR DRIVER 2"
+			(at 187.96 92.7099 0)
+			(show_name no)
+			(do_not_autoplace no)
+			(effects
+				(font
+					(size 1.27 1.27)
+				)
+				(justify left)
+			)
+		)
+		(property "Footprint" ""
+			(at 185.42 90.17 0)
+			(hide yes)
+			(show_name no)
+			(do_not_autoplace no)
+			(effects
+				(font
+					(size 1.27 1.27)
+				)
+			)
+		)
+		(property "Datasheet" ""
+			(at 185.42 90.17 0)
+			(hide yes)
+			(show_name no)
+			(do_not_autoplace no)
+			(effects
+				(font
+					(size 1.27 1.27)
+				)
+			)
+		)
+		(property "Description" "Generic connector, single row, 01x02, script generated (kicad-library-utils/schlib/autogen/connector/)"
+			(at 185.42 90.17 0)
+			(hide yes)
+			(show_name no)
+			(do_not_autoplace no)
+			(effects
+				(font
+					(size 1.27 1.27)
+				)
+			)
+		)
+		(pin "1"
+		)
+		(pin "2"
+		)
+		(instances
+			(project "Power Systems"
+				(path "/7d9b4746-b4fa-4905-9b55-f00e27d57e0a"
+					(reference "J2")
+					(unit 1)
+				)
+			)
+		)
+	)
+	(symbol
 		(lib_id "Connector_Generic:Conn_01x03")
 		(at 134.62 87.63 0)
@@
 	)
 	(symbol
+		(lib_id "Connector_Generic:Conn_01x02")
+		(at 185.42 105.41 0)
+		(unit 1)
+		(body_style 1)
+		(exclude_from_sim no)
+		(in_bom yes)
+		(on_board yes)
+		(in_pos_files yes)
+		(dnp no)
+		(fields_autoplaced yes)
+		(property "Reference" "J4"
+			(at 187.96 105.4099 0)
+			(show_name no)
+			(do_not_autoplace no)
+			(effects
+				(font
+					(size 1.27 1.27)
+				)
+				(justify left)
+			)
+		)
+		(property "Value" "MOTOR DRIVER 4"
+			(at 187.96 107.9499 0)
+			(show_name no)
+			(do_not_autoplace no)
+			(effects
+				(font
+					(size 1.27 1.27)
+				)
+				(justify left)
+			)
+		)
+		(property "Footprint" ""
+			(at 185.42 105.41 0)
+			(hide yes)
+			(show_name no)
+			(do_not_autoplace no)
+			(effects
+				(font
+					(size 1.27 1.27)
+				)
+			)
+		)
+		(property "Datasheet" ""
+			(at 185.42 105.41 0)
+			(hide yes)
+			(show_name no)
+			(do_not_autoplace no)
+			(effects
+				(font
+					(size 1.27 1.27)
+				)
+			)
+		)
+		(property "Description" "Generic connector, single row, 01x02, script generated (kicad-library-utils/schlib/autogen/connector/)"
+			(at 185.42 105.41 0)
+			(hide yes)
+			(show_name no)
+			(do_not_autoplace no)
+			(effects
+				(font
+					(size 1.27 1.27)
+				)
+			)
+		)
+		(pin "1"
+		)
+		(pin "2"
+		)
+		(instances
+			(project "Power Systems"
+				(path "/7d9b4746-b4fa-4905-9b55-f00e27d57e0a"
+					(reference "J4")
+					(unit 1)
+				)
+			)
+		)
+	)
+	(symbol
 		(lib_id "power:GND")
 		(at 31.75 57.15 0)
@@
 		(dnp no)
 		(fields_autoplaced yes)
-		(property "Reference" "J2"
+		(property "Reference" "J1"
 			(at 187.96 82.5499 0)
 			(show_name no)
@@
 			)
 		)
-		(property "Value" "Conn_01x02"
+		(property "Value" "MOTOR DRIVER 1"
 			(at 187.96 85.0899 0)
 			(show_name no)
@@
 			(project "Power Systems"
 				(path "/7d9b4746-b4fa-4905-9b55-f00e27d57e0a"
-					(reference "J2")
-					(unit 1)
-				)
+					(reference "J1")
+					(unit 1)
+				)

Commit message: Motor driver
---
Parts:
- removed J1: CURRENT SENSE, symbol Connector_Generic:Conn_01x03
- removed J1: MOTOR DRIVER 1, symbol Connector_Generic:Conn_01x02
- removed J2: MOTOR DRIVER 2, symbol Connector_Generic:Conn_01x02
- removed J3: MOTOR DRIVER 3, symbol Connector_Generic:Conn_01x02
- removed J4: MOTOR DRIVER 4, symbol Connector_Generic:Conn_01x02
- added J1: Conn_01x04, Package_TO_SOT_THT:TO-220-15_P2.54x5.08mm_StaggerOdd_Lead4.58mm_Vertical, symbol Connector_Generic:Conn_01x04
- added U2: CURRENT SENSE, symbol Connector_Generic:Conn_01x05
Connections:
- net GND: now also K1.2
- net VBATT: now also K1.4, K1.5, SW2.1, SW2.2
- net at F4.1: now also F2.1, F3.1, F5.1, U2.2 (Pin_2)
- net VMOTOR: now reaches K1.3
- net VMOTOR: now also U2.1 (Pin_1)
Other:
- moved on the sheet: F2, F3, F4, F5, K1, SW2

Commit message: f
Parts:
- added C2: C_Polarized 2200 uF 10V, symbol Device:C_Polarized
- added F6, F7: 5A Fuse, Package_LCC:PLCC-84_29.3x29.3mm_P1.27mm, symbol Device:Fuse
- added U1: INA226, Package_SO:TSSOP-10_3x3mm_P0.5mm, symbol Sensor_Energy:INA226
- added U4: 6V/5A Conv, Package_TO_SOT_THT:TO-220-15_P2.54x5.08mm_StaggerOdd_Lead4.58mm_Vertical, symbol Connector_Generic:Conn_01x04
- U3: renamed from J1; value Conn_01x04 -> 5V/5A Conv
Connections:
- net GND: now also U3.2 (Pin_2), C2.2, U1.7 (GND), U4.2 (Pin_2)
- net VBATT: now also U3.1 (Pin_1), U1.8 (Vbus), U4.1 (Pin_1); no longer C1.1, D1.1 (K)
- net at U3.3 (Pin_3): now also F6.1
- new net: C1.1, D1.1 (K), U1.10 (Vin+)
- new net: F7.1, U4.3 (Pin_3)
- new net: C2.1, F7.2
Other:
- moved on the sheet: F2, F3, F4, F5, K1, SW2, U2, U3

Commit message: gg
Parts:
- added F10, F8, F9: Polyfuse, Package_TO_SOT_SMD:SOT-223-3_TabPin2, symbol Device:Polyfuse
- added U5: LM317_SOT-223, Package_TO_SOT_SMD:SOT-223-3_TabPin2, symbol Regulator_Linear:LM317_SOT-223
Connections:
- net GND: now also F6.2, F10.1, F10.2, F8.1, F8.2, F9.1, F9.2, U5.1 (ADJ), U5.3 (VI)

Commit message: V1
Parts:
- added F11, F12, F13: Polyfuse, Package_TO_SOT_SMD:SOT-223-3_TabPin2, symbol Device:Polyfuse
Connections:
- net GND: now also F2.2, F3.2, F4.2, F5.2, F11.2, F12.2, F13.2
- net at C2.1, F7.2: now also F12.1, F13.1
- net at U5.2 (VO): now also F11.1
Other:
- moved on the sheet: F2, F3, F4, F5, U2
