File: Power Systems/Power Systems.kicad_sch (KiCad schematic)
At the start: 25 parts, among them K1 E-STOP RELAY 30A, SW1 MAIN DISCONECT - 30A, SW2 E-STOP NC, U1 INA226, U2 CURRENT SENSE, U3 5V/5A Conv, U4 6V/5A Conv, U5 LM317_SOT-223

Commit message: V1.5
New
Parts:
- added R1: Shunt Resistor, Package_DIP:DIP-8_W7.62mm, symbol Device:R
- added R2, R3: R, symbol Device:R
Connections:
- net GND: now also R2.2; no longer F10.1, F6.2, F8.1, F9.1, U5.1 (ADJ), U5.3 (VI)
- net VBATT: no longer K1.5, SW2.2
- net at F11.1, U5.2 (VO): now also R3.1
- net at C1.1, D1.1 (K), U1.10 (Vin+): now also R1.2
- net 3.3V OR 5V CDH Power Managament Component: now reaches U1.6 (VS)
- net at U1.9 (Vin-): now also R1.1
- new net: R2.1, R3.2, U5.1 (ADJ)
- new net: F10.1, F6.2, F8.1, F9.1, U5.3 (VI)
- new net: K1.5, SW2.2
Other:
- moved on the sheet: BT1
